Commit message: Reorganize packages

File: roboplan_examples/ur_robot_model/ur5_gripper.urdf (robot description, URDF)
Before this commit: robot ur5, 11 links, 10 joints
Links:
- link base_link: geometry collision mesh filename=package://roboplan_examples/ur_robot_model/meshes/collision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; visual mesh filename=package://roboplan_examples/ur_robot_model/meshes/visual/ba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
- link forearm_link: geometry collision mesh filename=package://roboplan_examples/ur_robot_model/meshes/collision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; visual mesh filename=package://roboplan_examples/ur_robot_model/meshes/visual/fo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
- link shoulder_link: geometry collision mesh filename=package://roboplan_examples/ur_robot_model/meshes/collision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; visual mesh filename=package://roboplan_examples/ur_robot_model/meshes/visual/sh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
- link upper_arm_link: geometry collision mesh filename=package://roboplan_examples/ur_robot_model/meshes/collision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; visual mesh filename=package://roboplan_examples/ur_robot_model/meshes/visual/up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
- link wrist_1_link: geometry collision mesh filename=package://roboplan_examples/ur_robot_model/meshes/collision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; visual mesh filename=package://roboplan_examples/ur_robot_model/meshes/visual/wr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
- link wrist_2_link: geometry collision mesh filename=package://roboplan_examples/ur_robot_model/meshes/collision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; visual mesh filename=package://roboplan_examples/ur_robot_model/meshes/visual/wr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
- link wrist_3_link: geometry collision mesh filename=package://roboplan_examples/ur_robot_model/meshes/collision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; visual mesh filename=package://roboplan_examples/ur_robot_model/meshes/visual/wr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
