Commit message: Split the ur_resources out to a separate library that can be included wherever

File: roboplan_examples/example_resources/ur_robot_model/ur5_gripper.urdf (robot description, URDF)
Before this commit: robot ur5, 11 links, 10 joints
Links:
- link base_link: geometry collision mesh filename=package://roboplan_example_resources/ur_robot_model/meshes/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; visual mesh filename=package://roboplan_example_resources/ur_robot_model/meshes/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
- link forearm_link: geometry collision mesh filename=package://roboplan_example_resources/ur_robot_model/meshes/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; visual mesh filename=package://roboplan_example_resources/ur_robot_model/meshes/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
- link shoulder_link: geometry collision mesh filename=package://roboplan_example_resources/ur_robot_model/meshes/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; visual mesh filename=package://roboplan_example_resources/ur_robot_model/meshes/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
- link upper_arm_link: geometry collision mesh filename=package://roboplan_example_resources/ur_robot_model/meshes/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; visual mesh filename=package://roboplan_example_resources/ur_robot_model/meshes/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
- link wrist_1_link: geometry collision mesh filename=package://roboplan_example_resources/ur_robot_model/meshes/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; visual mesh filename=package://roboplan_example_resources/ur_robot_model/meshes/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
- link wrist_2_link: geometry collision mesh filename=package://roboplan_example_resources/ur_robot_model/meshes/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; visual mesh filename=package://roboplan_example_resources/ur_robot_model/meshes/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
- link wrist_3_link: geometry collision mesh filename=package://roboplan_example_resources/ur_robot_model/meshes/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; visual mesh filename=package://roboplan_example_resources/ur_robot_model/meshes/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
