Commit message: Fix mesh paths

File: roboplan_example_models/models/ur_robot_model/ur5_gripper.urdf (robot description, URDF)
Before this commit: robot ur5, 11 links, 10 joints
Links:
- link base_link: geometry collision mesh filename=package://roboplan_example_models/models/ur_robot_model/mes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; visual mesh filename=package://roboplan_example_models/models/ur_robot_model/mes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
- link forearm_link: geometry collision mesh filename=package://roboplan_example_models/models/ur_robot_model/mes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; visual mesh filename=package://roboplan_example_models/models/ur_robot_model/mes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
- link shoulder_link: geometry collision mesh filename=package://roboplan_example_models/models/ur_robot_model/mes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; visual mesh filename=package://roboplan_example_models/models/ur_robot_model/mes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
- link upper_arm_link: geometry collision mesh filename=package://roboplan_example_models/models/ur_robot_model/mes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; visual mesh filename=package://roboplan_example_models/models/ur_robot_model/mes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
- link wrist_1_link: geometry collision mesh filename=package://roboplan_example_models/models/ur_robot_model/mes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; visual mesh filename=package://roboplan_example_models/models/ur_robot_model/mes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
- link wrist_2_link: geometry collision mesh filename=package://roboplan_example_models/models/ur_robot_model/mes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; visual mesh filename=package://roboplan_example_models/models/ur_robot_model/mes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
- link wrist_3_link: geometry collision mesh filename=package://roboplan_example_models/models/ur_robot_model/mes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; visual mesh filename=package://roboplan_example_models/models/ur_robot_model/mes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

Commit message: Add vanilla CMake workflow

File: roboplan_example_models/models/ur_robot_model/ur5_gripper.urdf (robot description, URDF)
Before this commit: robot ur5, 11 links, 10 joints
Links:
- link base_link: geometry collision mesh filename=package://ur_robot_model/meshes/collision/base.stl; visual mesh filename=package://ur_robot_model/meshes/visual/base.dae
- link forearm_link: geometry collision mesh filename=package://ur_robot_model/meshes/collision/forearm.stl; visual mesh filename=package://ur_robot_model/meshes/visual/forearm.dae
- link shoulder_link: geometry collision mesh filename=package://ur_robot_model/meshes/collision/shoulder.stl; visual mesh filename=package://ur_robot_model/meshes/visual/shoulder.dae
- link upper_arm_link: geometry collision mesh filename=package://ur_robot_model/meshes/collision/upperarm.stl; visual mesh filename=package://ur_robot_model/meshes/visual/upperarm.dae
- link wrist_1_link: geometry collision mesh filename=package://ur_robot_model/meshes/collision/wrist1.stl; visual mesh filename=package://ur_robot_model/meshes/visual/wrist1.dae
- link wrist_2_link: geometry collision mesh filename=package://ur_robot_model/meshes/collision/wrist2.stl; visual mesh filename=package://ur_robot_model/meshes/visual/wrist2.dae
- link wrist_3_link: geometry collision mesh filename=package://ur_robot_model/meshes/collision/wrist3.stl; visual mesh filename=package://ur_robot_model/meshes/visual/wrist3.dae
