Commit message: Fixes thanks to eho

File: roboplan_example_models/models/kinova_robot_model/kinova_robotiq.urdf (robot description, URDF)
Before this commit: robot kinova_robotiq, 19 links, 18 joints
Links:
- link robotiq_85_base_link: geometry collision mesh filename=package://kinova_robot_model/meshes/collision/robotiq_base.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; visual mesh filename=package://kinova_robot_model/meshes/visual/robotiq_base.dae
- link robotiq_85_left_finger_link: geometry collision mesh filename=package://kinova_robot_model/meshes/collision/left_finger.s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; visual mesh filename=package://kinova_robot_model/meshes/visual/left_finger.dae
- link robotiq_85_left_finger_tip_link: geometry collision mesh filename=package://kinova_robot_model/meshes/collision/left_finger_t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; visual mesh filename=package://kinova_robot_model/meshes/visual/left_finger_tip.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
- link robotiq_85_left_inner_knuckle_link: geometry collision mesh filename=package://kinova_robot_model/meshes/collision/left_inner_kn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; visual mesh filename=package://kinova_robot_model/meshes/visual/left_inner_knuck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
- link robotiq_85_left_knuckle_link: geometry collision mesh filename=package://kinova_robot_model/meshes/collision/left_knuckle.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; visual mesh filename=package://kinova_robot_model/meshes/visual/left_knuckle.dae
- link robotiq_85_right_finger_link: geometry collision mesh filename=package://kinova_robot_model/meshes/collision/right_finger.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; visual mesh filename=package://kinova_robot_model/meshes/visual/right_finger.dae
- link robotiq_85_right_finger_tip_link: geometry collision mesh filename=package://kinova_robot_model/meshes/collision/right_finger_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; visual mesh filename=package://kinova_robot_model/meshes/visual/right_finger_tip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
- link robotiq_85_right_inner_knuckle_link: geometry collision mesh filename=package://kinova_robot_model/meshes/collision/right_inner_k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; visual mesh filename=package://kinova_robot_model/meshes/visual/right_inner_knuc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
- link robotiq_85_right_knuckle_link: geometry collision mesh filename=package://kinova_robot_model/meshes/collision/right_knuckle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; visual mesh filename=package://kinova_robot_model/meshes/visual/right_knuckle.dae
