Commit message: Make example models locatable in Rviz

File: roboplan_example_models/models/franka_robot_model/fr3.xacro (robot description, xacro)
@@ -13,10 +13,10 @@
       <visual name="${prefix}fr3_link0_visual">
         <geometry>
-          <mesh filename="package://franka_robot_model/meshes/visual/link0.dae"/>
+          <mesh filename="package://roboplan_example_models/models/franka_robot_model/meshes/visual/link0.dae"/>
         </geometry>
       </visual>
       <collision name="${prefix}fr3_link0_collision">
         <geometry>
-          <mesh filename="package://franka_robot_model/meshes/collision/link0.stl"/>
+          <mesh filename="package://roboplan_example_models/models/franka_robot_model/meshes/collision/link0.stl"/>
         </geometry>
       </collision>
@@ -30,10 +30,10 @@
       <visual name="${prefix}fr3_link1_visual">
         <geometry>
-          <mesh filename="package://franka_robot_model/meshes/visual/link1.dae"/>
+          <mesh filename="package://roboplan_example_models/models/franka_robot_model/meshes/visual/link1.dae"/>
         </geometry>
       </visual>
       <collision name="${prefix}fr3_link1_collision">
         <geometry>
-          <mesh filename="package://franka_robot_model/meshes/collision/link1.stl"/>
+          <mesh filename="package://roboplan_example_models/models/franka_robot_model/meshes/collision/link1.stl"/>
         </geometry>
       </collision>
@@ -56,10 +56,10 @@
       <visual name="${prefix}fr3_link2_visual">
         <geometry>
-          <mesh filename="package://franka_robot_model/meshes/visual/link2.dae"/>
+          <mesh filename="package://roboplan_example_models/models/franka_robot_model/meshes/visual/link2.dae"/>
         </geometry>
       </visual>
       <collision name="${prefix}fr3_link2_collision">
         <geometry>
-          <mesh filename="package://franka_robot_model/meshes/collision/link2.stl"/>
+          <mesh filename="package://roboplan_example_models/models/franka_robot_model/meshes/collision/link2.stl"/>
         </geometry>
       </collision>
@@ -82,10 +82,10 @@
       <visual name="${prefix}fr3_link3_visual">
         <geometry>
-          <mesh filename="package://franka_robot_model/meshes/visual/link3.dae"/>
+          <mesh filename="package://roboplan_example_models/models/franka_robot_model/meshes/visual/link3.dae"/>
         </geometry>
       </visual>
       <collision name="${prefix}fr3_link3_collision">
         <geometry>
-          <mesh filename="package://franka_robot_model/meshes/collision/link3.stl"/>
+          <mesh filename="package://roboplan_example_models/models/franka_robot_model/meshes/collision/link3.stl"/>
         </geometry>
       </collision>
@@ -108,10 +108,10 @@
       <visual name="${prefix}fr3_link4_visual">
         <geometry>
-          <mesh filename="package://franka_robot_model/meshes/visual/link4.dae"/>
+          <mesh filename="package://roboplan_example_models/models/franka_robot_model/meshes/visual/link4.dae"/>
         </geometry>
       </visual>
       <collision name="${prefix}fr3_link4_collision">
         <geometry>
-          <mesh filename="package://franka_robot_model/meshes/collision/link4.stl"/>
+          <mesh filename="package://roboplan_example_models/models/franka_robot_model/meshes/collision/link4.stl"/>
         </geometry>
       </collision>
@@ -134,10 +134,10 @@
       <visual name="${prefix}fr3_link5_visual">
         <geometry>
-          <mesh filename="package://franka_robot_model/meshes/visual/link5.dae"/>
+          <mesh filename="package://roboplan_example_models/models/franka_robot_model/meshes/visual/link5.dae"/>
         </geometry>
       </visual>
       <collision name="${prefix}fr3_link5_collision">
         <geometry>
-          <mesh filename="package://franka_robot_model/meshes/collision/link5.stl"/>
+          <mesh filename="package://roboplan_example_models/models/franka_robot_model/meshes/collision/link5.stl"/>
         </geometry>
       </collision>
@@ -160,10 +160,10 @@
       <visual name="${prefix}fr3_link6_visual">
         <geometry>
-          <mesh filename="package://franka_robot_model/meshes/visual/link6.dae"/>
+          <mesh filename="package://roboplan_example_models/models/franka_robot_model/meshes/visual/link6.dae"/>
         </geometry>
       </visual>
       <collision name="${prefix}fr3_link6_collision">
         <geometry>
-          <mesh filename="package://franka_robot_model/meshes/collision/link6.stl"/>
+          <mesh filename="package://roboplan_example_models/models/franka_robot_model/meshes/collision/link6.stl"/>
         </geometry>
       </collision>
@@ -186,10 +186,10 @@
       <visual name="${prefix}fr3_link7_visual">
         <geometry>
-          <mesh filename="package://franka_robot_model/meshes/visual/link7.dae"/>
+          <mesh filename="package://roboplan_example_models/models/franka_robot_model/meshes/visual/link7.dae"/>
         </geometry>
       </visual>
       <collision name="${prefix}fr3_link7_collision">
         <geometry>
-          <mesh filename="package://franka_robot_model/meshes/collision/link7.stl"/>
+          <mesh filename="package://roboplan_example_models/models/franka_robot_model/meshes/collision/link7.stl"/>
         </geometry>
       </collision>
@@ -223,10 +223,10 @@
       <visual name="${prefix}fr3_hand_visual">
         <geometry>
-          <mesh filename="package://franka_robot_model/meshes/visual/hand.dae"/>
+          <mesh filename="package://roboplan_example_models/models/franka_robot_model/meshes/visual/hand.dae"/>
         </geometry>
       </visual>
       <collision name="${prefix}fr3_hand_collision">
         <geometry>
-          <mesh filename="package://franka_robot_model/meshes/collision/hand.stl"/>
+          <mesh filename="package://roboplan_example_models/models/franka_robot_model/meshes/collision/hand.stl"/>
         </geometry>
       </collision>
@@ -247,5 +247,5 @@
       <visual name="${prefix}fr3_leftfinger_visual">
         <geometry>
-          <mesh filename="package://franka_robot_model/meshes/visual/finger.dae"/>
+          <mesh filename="package://roboplan_example_models/models/franka_robot_model/meshes/visual/finger.dae"/>
         </geometry>
       </visual>
@@ -288,5 +288,5 @@
         <origin rpy="0 0 0" xyz="0 0 0"/>
         <geometry>
-          <mesh filename="package://franka_robot_model/meshes/visual/finger.dae"/>
+          <mesh filename="package://roboplan_example_models/models/franka_robot_model/meshes/visual/finger.dae"/>
         </geometry>
       </visual>

File: roboplan_example_models/models/kinova_robot_model/kinova_robotiq.urdf (robot description, URDF)
Before this commit: robot kinova_robotiq, 19 links, 18 joints
Links:
- link base_link: geometry collision mesh filename=package://roboplan_example_models/models/kinova_robot_model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; visual mesh filename=package://roboplan_example_models/models/kinova_robot_model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
- link bracelet_link: geometry collision mesh filename=package://roboplan_example_models/models/kinova_robot_model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; visual mesh filename=package://roboplan_example_models/models/kinova_robot_model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
- link forearm_link: geometry collision mesh filename=package://roboplan_example_models/models/kinova_robot_model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; visual mesh filename=package://roboplan_example_models/models/kinova_robot_model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
- link half_arm_1_link: geometry collision mesh filename=package://roboplan_example_models/models/kinova_robot_model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; visual mesh filename=package://roboplan_example_models/models/kinova_robot_model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
- link half_arm_2_link: geometry collision mesh filename=package://roboplan_example_models/models/kinova_robot_model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; visual mesh filename=package://roboplan_example_models/models/kinova_robot_model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
- link robotiq_85_base_link: geometry collision mesh filename=package://roboplan_example_models/models/kinova_robot_model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; visual mesh filename=package://roboplan_example_models/models/kinova_robot_model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
- link robotiq_85_left_finger_link: geometry collision mesh filename=package://roboplan_example_models/models/kinova_robot_model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; visual mesh filename=package://roboplan_example_models/models/kinova_robot_model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
- link robotiq_85_left_finger_tip_link: geometry collision mesh filename=package://roboplan_example_models/models/kinova_robot_model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; visual mesh filename=package://roboplan_example_models/models/kinova_robot_model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
- link robotiq_85_left_inner_knuckle_link: geometry collision mesh filename=package://roboplan_example_models/models/kinova_robot_model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; visual mesh filename=package://roboplan_example_models/models/kinova_robot_model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
- link robotiq_85_left_knuckle_link: geometry collision mesh filename=package://roboplan_example_models/models/kinova_robot_model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; visual mesh filename=package://roboplan_example_models/models/kinova_robot_model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
- link robotiq_85_right_finger_link: geometry collision mesh filename=package://roboplan_example_models/models/kinova_robot_model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; visual mesh filename=package://roboplan_example_models/models/kinova_robot_model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
- link robotiq_85_right_finger_tip_link: geometry collision mesh filename=package://roboplan_example_models/models/kinova_robot_model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; visual mesh filename=package://roboplan_example_models/models/kinova_robot_model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
- link robotiq_85_right_inner_knuckle_link: geometry collision mesh filename=package://roboplan_example_models/models/kinova_robot_model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; visual mesh filename=package://roboplan_example_models/models/kinova_robot_model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
- link robotiq_85_right_knuckle_link: geometry collision mesh filename=package://roboplan_example_models/models/kinova_robot_model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; visual mesh filename=package://roboplan_example_models/models/kinova_robot_model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
- link shoulder_link: geometry collision mesh filename=package://roboplan_example_models/models/kinova_robot_model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; visual mesh filename=package://roboplan_example_models/models/kinova_robot_model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
- link spherical_wrist_1_link: geometry collision mesh filename=package://roboplan_example_models/models/kinova_robot_model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; visual mesh filename=package://roboplan_example_models/models/kinova_robot_model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
- link spherical_wrist_2_link: geometry collision mesh filename=package://roboplan_example_models/models/kinova_robot_model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; visual mesh filename=package://roboplan_example_models/models/kinova_robot_model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

File: roboplan_example_models/models/ur_robot_model/ur5_gripper.urdf (robot description, URDF)
Before this commit: robot ur5, 11 links, 10 joints
Links:
- link base_link: geometry collision mesh filename=package://roboplan_example_models/models/ur_robot_model/mes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; visual mesh filename=package://roboplan_example_models/models/ur_robot_model/mes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
- link forearm_link: geometry collision mesh filename=package://roboplan_example_models/models/ur_robot_model/mes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; visual mesh filename=package://roboplan_example_models/models/ur_robot_model/mes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
- link shoulder_link: geometry collision mesh filename=package://roboplan_example_models/models/ur_robot_model/mes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; visual mesh filename=package://roboplan_example_models/models/ur_robot_model/mes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
- link upper_arm_link: geometry collision mesh filename=package://roboplan_example_models/models/ur_robot_model/mes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; visual mesh filename=package://roboplan_example_models/models/ur_robot_model/mes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
- link wrist_1_link: geometry collision mesh filename=package://roboplan_example_models/models/ur_robot_model/mes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; visual mesh filename=package://roboplan_example_models/models/ur_robot_model/mes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
- link wrist_2_link: geometry collision mesh filename=package://roboplan_example_models/models/ur_robot_model/mes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; visual mesh filename=package://roboplan_example_models/models/ur_robot_model/mes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
- link wrist_3_link: geometry collision mesh filename=package://roboplan_example_models/models/ur_robot_model/mes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; visual mesh filename=package://roboplan_example_models/models/ur_robot_model/mes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

Commit message: Add ros2_control tags to Franka xacro

File: roboplan_example_models/models/franka_robot_model/fr3.xacro (robot description, xacro)
@@ -342,4 +342,117 @@
       <dynamics damping="0.3"/>
     </joint>
+  <!-- ros2_control setup for mock hardware -->
+  <ros2_control name="${prefix}name" type="system">
+    <hardware>
+      <plugin>mock_components/GenericSystem</plugin>
+      <param name="mock_sensor_commands">false</param>
+      <param name="state_following_offset">0.0</param>
+      <param name="calculate_dynamics">true</param>
+    </hardware>
+    <joint name="${prefix}fr3_joint1">
+      <command_interface name="position"/>
+      <command_interface name="velocity"/>
+      <state_interface name="position">
+        <param name="initial_value">0.0</param>
+      </state_interface>
+      <state_interface name="velocity">
+        <param name="initial_value">0.0</param>
+      </state_interface>
+      <state_interface name="effort">
+        <param name="initial_value">0.0</param>
+      </state_interface>
+    </joint>
+    <joint name="${prefix}fr3_joint2">
+      <command_interface name="position"/>
+      <command_interface name="velocity"/>
+      <state_interface name="position">
+        <param name="initial_value">${-pi/4}</param>
+      </state_interface>
+      <state_interface name="velocity">
+        <param name="initial_value">0.0</param>
+      </state_interface>
+      <state_interface name="effort">
+        <param name="initial_value">0.0</param>
+      </state_interface>
+    </joint>
+    <joint name="${prefix}fr3_joint3">
+      <command_interface name="position"/>
+      <command_interface name="velocity"/>
+      <state_interface name="position">
+        <param name="initial_value">0.0</param>
+      </state_interface>
+      <state_interface name="velocity">
+        <param name="initial_value">0.0</param>
+      </state_interface>
+      <state_interface name="effort">
+        <param name="initial_value">0.0</param>
+      </state_interface>
+    </joint>
+    <joint name="${prefix}fr3_joint4">
+      <command_interface name="position"/>
+      <command_interface name="velocity"/>
+      <state_interface name="position">
+        <param name="initial_value">${-3*pi/4}</param>
+      </state_interface>
+      <state_interface name="velocity">
+        <param name="initial_value">0.0</param>
+      </state_interface>
+      <state_interface name="effort">
+        <param name="initial_value">0.0</param>
+      </state_interface>
+    </joint>
+    <joint name="${prefix}fr3_joint5">
+      <command_interface name="position"/>
+      <command_interface name="velocity"/>
+      <state_interface name="position">
+        <param name="initial_value">0.0</param>
+      </state_interface>
+      <state_interface name="velocity">
+        <param name="initial_value">0.0</param>
+      </state_interface>
+      <state_interface name="effort">
+        <param name="initial_value">0.0</param>
+      </state_interface>
+    </joint>
+    <joint name="${prefix}fr3_joint6">
+      <command_interface name="position"/>
+      <command_interface name="velocity"/>
+      <state_interface name="position">
+        <param name="initial_value">${pi/2}</param>
+      </state_interface>
+      <state_interface name="velocity">
+        <param name="initial_value">0.0</param>
+      </state_interface>
+      <state_interface name="effort">
+        <param name="initial_value">0.0</param>
+      </state_interface>
+    </joint>
+    <joint name="${prefix}fr3_joint7">
+      <command_interface name="position"/>
+      <command_interface name="velocity"/>
+      <state_interface name="position">
+        <param name="initial_value">${pi/4}</param>
+      </state_interface>
+      <state_interface name="velocity">
+        <param name="initial_value">0.0</param>
+      </state_interface>
+      <state_interface name="effort">
+        <param name="initial_value">0.0</param>
+      </state_interface>
+    </joint>
+    <joint name="${prefix}fr3_finger_joint1">
+      <command_interface name="position"/>
+      <command_interface name="velocity"/>
+      <state_interface name="position">
+        <param name="initial_value">0.0</param>
+      </state_interface>
+      <state_interface name="velocity">
+        <param name="initial_value">0.0</param>
+      </state_interface>
+      <state_interface name="effort">
+        <param name="initial_value">0.0</param>
+      </state_interface>
+    </joint>
+  </ros2_control>
   </xacro:macro>
 </robot>
