Commit message: increase velocity limit for rrt example to follow path

File: roboplan_example_models/models/stretch4_robot_model/stretch4_sg4.urdf (robot description, URDF)
Before this commit: robot stretch, 55 links, 54 joints
Joints:
- joint arm_l1_joint: limit lower=0 upper=0.13 effort=0 velocity=0 -> lower=0 upper=0.13 effort=0 velocity=0.05
- joint arm_l2_joint: limit lower=0 upper=0.13 effort=0 velocity=0 -> lower=0 upper=0.13 effort=0 velocity=0.05
- joint arm_l3_joint: limit lower=0 upper=0.13 effort=0 velocity=0 -> lower=0 upper=0.13 effort=0 velocity=0.05
- joint arm_l4_joint: limit lower=0 upper=0.13 effort=0 velocity=0 -> lower=0 upper=0.13 effort=0 velocity=0.05
- joint gripper_finger_left_joint: limit lower=0.0 upper=0.5 effort=0 velocity=0 -> lower=0.0 upper=0.5 effort=0 velocity=0.5
- joint gripper_finger_right_joint: limit lower=0.0 upper=0.5 effort=0 velocity=0 -> lower=0.0 upper=0.5 effort=0 velocity=0.5
- joint lift_joint: limit lower=0 upper=1.2 effort=0 velocity=0 -> lower=0 upper=1.2 effort=0 velocity=0.15
- joint wrist_pitch_joint: limit lower=-4.276 upper=1.135 effort=0 velocity=0 -> lower=-4.276 upper=1.135 effort=0 velocity=1.0
- joint wrist_roll_joint: limit lower=-1.135 upper=4.276 effort=0 velocity=0 -> lower=-1.135 upper=4.276 effort=0 velocity=1.0
- joint wrist_yaw_joint: limit lower=-1.135 upper=4.276 effort=0 velocity=0 -> lower=-1.135 upper=4.276 effort=0 velocity=1.0

Commit message: use plannar joint instead of 1DOF joints

File: roboplan_example_models/models/stretch4_robot_model/stretch4_sg4.urdf (robot description, URDF)
Before this commit: robot stretch, 55 links, 54 joints
Links:
- removed link base_xy_link
- removed link base_yaw_link
Joints:
- removed joint base_x_joint
- removed joint base_y_joint
- removed joint base_yaw_joint
- added joint mobile_base_planar_joint: type planar, parent base_footprint, child base_link, origin xyz=0 0 0.028 rpy=0 0 0, axis 0 0 1, limit lower=-2.0 upper=2.0 effort=100 velocity=0.5
